File: miniPCI_ZIF48.kicad_sch (KiCad schematic)
At the start: 6 parts

Commit message: Add footprints for ZIF-48 & mini-PCI-Type-III
Parts:
- ZIF-48P1: footprint (none) -> DIP-48_W15.24mm:DIP-48_W15.24mm_Socket
- mPCIE-62P1: footprint (none) -> mini_PCI_Type_III_female_Socket:MINIPCI_TYPE_IIIA
Changed lines of the file:
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@@
 			)
 		)
-		(property "Footprint" ""
-			(at 100.584 24.13 0)
+		(property "Footprint" "DIP-48_W15.24mm:DIP-48_W15.24mm_Socket"
+			(at 109.474 13.462 0)
 			(effects
 				(font
@@
 			)
 		)
-		(property "Footprint" ""
+		(property "Footprint" "mini_PCI_Type_III_female_Socket:MINIPCI_TYPE_IIIA"
 			(at 29.21 59.69 0)
 			(effects

Commit message: Passed all DRCs/PCB_Editor
Parts:
- C1, C2, C3, C4: footprint Capacitor_SMD:C_1206_3216Metric -> Capacitor_THT:C_Axial_L3.8mm_D2.6mm_P7.50mm_Horizontal

Commit message: Refine into only 2-layers design, both copper filled.
Parts:
- C1, C2, C3, C4: footprint Capacitor_THT:C_Axial_L3.8mm_D2.6mm_P7.50mm_Horizontal -> Capacitor_SMD:C_1206_3216Metric
Changed lines of the file:
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@@
 			)
 		)
-		(property "Footprint" "Capacitor_THT:C_Axial_L3.8mm_D2.6mm_P7.50mm_Horizontal"
+		(property "Footprint" "Capacitor_SMD:C_1206_3216Metric"
 			(at 65.0748 99.06 0)
 			(effects
@@
 			)
 		)
-		(property "Footprint" "Capacitor_THT:C_Axial_L3.8mm_D2.6mm_P7.50mm_Horizontal"
+		(property "Footprint" "Capacitor_SMD:C_1206_3216Metric"
 			(at 38.4048 99.06 0)
 			(effects
@@
 			)
 		)
-		(property "Footprint" "Capacitor_THT:C_Axial_L3.8mm_D2.6mm_P7.50mm_Horizontal"
+		(property "Footprint" "Capacitor_SMD:C_1206_3216Metric"
 			(at 157.1752 86.36 0)
 			(effects
@@
 			)
 		)
-		(property "Footprint" "Capacitor_THT:C_Axial_L3.8mm_D2.6mm_P7.50mm_Horizontal"
+		(property "Footprint" "Capacitor_SMD:C_1206_3216Metric"
 			(at 134.3152 86.36 0)
 			(effects
